Commit message: fixup

File: trajopt/test/data/arm_around_table.urdf (robot description, URDF)
Before this commit: robot pr2, 89 links, 88 joints
Links:
- link table_link: geometry collision mesh filename=package://trajopt/test/data/meshes/Table.stl; visual mesh filename=package://trajopt/test/data/meshes/Table.stl

File: trajopt/test/data/boxbot.xacro (robot description, xacro)
@@ -1,6 +1,6 @@
 <?xml version="1.0" ?>
 <robot name="boxbot" xmlns:xacro="http://ros.org/wiki/xacro">
-  <xacro:include filename="$(find trajopt_test_support)/urdf/boxbot_macro.xacro"/>
-  <xacro:include filename="$(find trajopt_test_support)/urdf/box_1m_macro.xacro"/>
+  <xacro:include filename="$(find trajopt)/test/data/boxbot_macro.xacro"/>
+  <xacro:include filename="$(find trajopt)/test/data/box_1m_macro.xacro"/>
   <xacro:boxbot prefix=""/>
   <xacro:box_1m prefix="test_"/>

File: trajopt/test/data/boxbot_world.xacro (robot description, xacro)
@@ -1,5 +1,5 @@
 <?xml version="1.0" ?>
 <robot name="boxbot" xmlns:xacro="http://ros.org/wiki/xacro">
-  <xacro:include filename="$(find trajopt_test_support)/urdf/boxbot_macro.xacro"/>
+  <xacro:include filename="$(find trajopt)/test/data/boxbot_macro.xacro"/>
   <xacro:boxbot prefix=""/>
 </robot>

Commit message: Add console_bridge and remove rosconsole and fix tests

File: trajopt/test/data/arm_around_table.urdf (robot description, URDF)
Before this commit: robot pr2, 89 links, 88 joints
Links:
- link base_link: geometry collision mesh filename=package://trajopt/test/data/pr2/meshes/base_v0/base_L.stl; visual mesh filename=package://trajopt/test/data/pr2/meshes/base_v0/base.dae
- link bl_caster_l_wheel_link: geometry collision cylinder length=0.034 radius=0.074792; visual mesh filename=package://trajopt/test/data/pr2/meshes/base_v0/wheel.dae
- link bl_caster_r_wheel_link: geometry collision cylinder length=0.034 radius=0.074792; visual mesh filename=package://trajopt/test/data/pr2/meshes/base_v0/wheel.dae
- link bl_caster_rotation_link: geometry collision mesh filename=package://trajopt/test/data/pr2/meshes/base_v0/caster_L.stl; visual mesh filename=package://trajopt/test/data/pr2/meshes/base_v0/caster.stl
- link br_caster_l_wheel_link: geometry collision cylinder length=0.034 radius=0.074792; visual mesh filename=package://trajopt/test/data/pr2/meshes/base_v0/wheel.dae
- link br_caster_r_wheel_link: geometry collision cylinder length=0.034 radius=0.074792; visual mesh filename=package://trajopt/test/data/pr2/meshes/base_v0/wheel.dae
- link br_caster_rotation_link: geometry collision mesh filename=package://trajopt/test/data/pr2/meshes/base_v0/caster_L.stl; visual mesh filename=package://trajopt/test/data/pr2/meshes/base_v0/caster.stl
- link fl_caster_l_wheel_link: geometry collision cylinder length=0.034 radius=0.074792; visual mesh filename=package://trajopt/test/data/pr2/meshes/base_v0/wheel.dae
- link fl_caster_r_wheel_link: geometry collision cylinder length=0.034 radius=0.074792; visual mesh filename=package://trajopt/test/data/pr2/meshes/base_v0/wheel.dae
- link fl_caster_rotation_link: geometry collision mesh filename=package://trajopt/test/data/pr2/meshes/base_v0/caster_L.stl; visual mesh filename=package://trajopt/test/data/pr2/meshes/base_v0/caster.stl
- link fr_caster_l_wheel_link: geometry collision cylinder length=0.034 radius=0.074792; visual mesh filename=package://trajopt/test/data/pr2/meshes/base_v0/wheel.dae
- link fr_caster_r_wheel_link: geometry collision cylinder length=0.034 radius=0.074792; visual mesh filename=package://trajopt/test/data/pr2/meshes/base_v0/wheel.dae
- link fr_caster_rotation_link: geometry collision mesh filename=package://trajopt/test/data/pr2/meshes/base_v0/caster_L.stl; visual mesh filename=package://trajopt/test/data/pr2/meshes/base_v0/caster.stl
- link head_pan_link: geometry collision mesh filename=package://trajopt/test/data/pr2/meshes/head_v0/head_pan_L.s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; visual mesh filename=package://trajopt/test/data/pr2/meshes/head_v0/head_pan.dae
- link head_tilt_link: geometry collision mesh filename=package://trajopt/test/data/pr2/meshes/head_v0/head_tilt_L.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; visual mesh filename=package://trajopt/test/data/pr2/meshes/head_v0/head_tilt.dae
- link l_elbow_flex_link: geometry collision mesh filename=package://trajopt/test/data/pr2/meshes/upper_arm_v0/elbow_f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; visual mesh filename=package://trajopt/test/data/pr2/meshes/upper_arm_v0/elbow_f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
- link l_forearm_link: geometry collision mesh filename=package://trajopt/test/data/pr2/meshes/forearm_v0/forearm.s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; visual mesh filename=package://trajopt/test/data/pr2/meshes/forearm_v0/forearm.d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
- link l_forearm_roll_link: geometry collision mesh filename=package://trajopt/test/data/pr2/meshes/upper_arm_v0/forearm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; visual mesh filename=package://trajopt/test/data/pr2/meshes/upper_arm_v0/forearm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
- link l_gripper_l_finger_link: geometry collision mesh filename=package://trajopt/test/data/pr2/meshes/gripper_v0/l_finger.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; visual mesh filename=package://trajopt/test/data/pr2/meshes/gripper_v0/l_finger.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
- link l_gripper_l_finger_tip_link: geometry collision mesh filename=package://trajopt/test/data/pr2/meshes/gripper_v0/l_finger_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; visual mesh filename=package://trajopt/test/data/pr2/meshes/gripper_v0/l_finger_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
- link l_gripper_palm_link: geometry collision mesh filename=package://trajopt/test/data/pr2/meshes/gripper_v0/gripper_p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; visual mesh filename=package://trajopt/test/data/pr2/meshes/gripper_v0/gripper_p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
- link l_gripper_r_finger_link: geometry collision mesh filename=package://trajopt/test/data/pr2/meshes/gripper_v0/l_finger.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; visual mesh filename=package://trajopt/test/data/pr2/meshes/gripper_v0/l_finger.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
- link l_gripper_r_finger_tip_link: geometry collision mesh filename=package://trajopt/test/data/pr2/meshes/gripper_v0/l_finger_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; visual mesh filename=package://trajopt/test/data/pr2/meshes/gripper_v0/l_finger_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
- link l_shoulder_lift_link: geometry collision mesh filename=package://trajopt/test/data/pr2/meshes/shoulder_v0/shoulder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; visual mesh filename=package://trajopt/test/data/pr2/meshes/shoulder_v0/shoulder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
- link l_shoulder_pan_link: geometry collision mesh filename=package://trajopt/test/data/pr2/meshes/shoulder_v0/shoulder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; visual mesh filename=package://trajopt/test/data/pr2/meshes/shoulder_v0/shoulder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
- link l_upper_arm_link: geometry collision mesh filename=package://trajopt/test/data/pr2/meshes/upper_arm_v0/upper_a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; visual mesh filename=package://trajopt/test/data/pr2/meshes/upper_arm_v0/upper_a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
- link l_upper_arm_roll_link: geometry collision mesh filename=package://trajopt/test/data/pr2/meshes/shoulder_v0/upper_ar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; visual mesh filename=package://trajopt/test/data/pr2/meshes/shoulder_v0/upper_ar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
- link l_wrist_flex_link: geometry collision mesh filename=package://trajopt/test/data/pr2/meshes/forearm_v0/wrist_fle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; visual mesh filename=package://trajopt/test/data/pr2/meshes/forearm_v0/wrist_fle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
- link l_wrist_roll_link: geometry collision mesh filename=package://trajopt/test/data/pr2/meshes/forearm_v0/wrist_rol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; visual mesh filename=package://trajopt/test/data/pr2/meshes/forearm_v0/wrist_rol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
- link laser_tilt_mount_link: geometry collision mesh filename=package://trajopt/test/data/pr2/meshes/tilting_laser_v0/til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; visual mesh filename=package://trajopt/test/data/pr2/meshes/tilting_laser_v0/til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
- link r_elbow_flex_link: geometry collision mesh filename=package://trajopt/test/data/pr2/meshes/upper_arm_v0/elbow_f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; visual mesh filename=package://trajopt/test/data/pr2/meshes/upper_arm_v0/elbow_f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
- link r_forearm_link: geometry collision mesh filename=package://trajopt/test/data/pr2/meshes/forearm_v0/forearm.s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; visual mesh filename=package://trajopt/test/data/pr2/meshes/forearm_v0/forearm.d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
- link r_forearm_roll_link: geometry collision mesh filename=package://trajopt/test/data/pr2/meshes/upper_arm_v0/forearm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; visual mesh filename=package://trajopt/test/data/pr2/meshes/upper_arm_v0/forearm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
- link r_gripper_l_finger_link: geometry collision mesh filename=package://trajopt/test/data/pr2/meshes/gripper_v0/l_finger.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; visual mesh filename=package://trajopt/test/data/pr2/meshes/gripper_v0/l_finger.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
- link r_gripper_l_finger_tip_link: geometry collision mesh filename=package://trajopt/test/data/pr2/meshes/gripper_v0/l_finger_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; visual mesh filename=package://trajopt/test/data/pr2/meshes/gripper_v0/l_finger_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
- link r_gripper_palm_link: geometry collision mesh filename=package://trajopt/test/data/pr2/meshes/gripper_v0/gripper_p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; visual mesh filename=package://trajopt/test/data/pr2/meshes/gripper_v0/gripper_p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
- link r_gripper_r_finger_link: geometry collision mesh filename=package://trajopt/test/data/pr2/meshes/gripper_v0/l_finger.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; visual mesh filename=package://trajopt/test/data/pr2/meshes/gripper_v0/l_finger.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
- link r_gripper_r_finger_tip_link: geometry collision mesh filename=package://trajopt/test/data/pr2/meshes/gripper_v0/l_finger_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; visual mesh filename=package://trajopt/test/data/pr2/meshes/gripper_v0/l_finger_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
- link r_shoulder_lift_link: geometry collision mesh filename=package://trajopt/test/data/pr2/meshes/shoulder_v0/shoulder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; visual mesh filename=package://trajopt/test/data/pr2/meshes/shoulder_v0/shoulder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
- link r_shoulder_pan_link: geometry collision mesh filename=package://trajopt/test/data/pr2/meshes/shoulder_v0/shoulder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; visual mesh filename=package://trajopt/test/data/pr2/meshes/shoulder_v0/shoulder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
- link r_upper_arm_link: geometry collision mesh filename=package://trajopt/test/data/pr2/meshes/upper_arm_v0/upper_a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; visual mesh filename=package://trajopt/test/data/pr2/meshes/upper_arm_v0/upper_a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
- link r_upper_arm_roll_link: geometry collision mesh filename=package://trajopt/test/data/pr2/meshes/shoulder_v0/upper_ar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; visual mesh filename=package://trajopt/test/data/pr2/meshes/shoulder_v0/upper_ar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
- link r_wrist_flex_link: geometry collision mesh filename=package://trajopt/test/data/pr2/meshes/forearm_v0/wrist_fle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; visual mesh filename=package://trajopt/test/data/pr2/meshes/forearm_v0/wrist_fle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
- link r_wrist_roll_link: geometry collision mesh filename=package://trajopt/test/data/pr2/meshes/forearm_v0/wrist_rol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; visual mesh filename=package://trajopt/test/data/pr2/meshes/forearm_v0/wrist_rol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
- link torso_lift_link: geometry collision mesh filename=package://trajopt/test/data/pr2/meshes/torso_v0/torso_lift_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; visual mesh filename=package://trajopt/test/data/pr2/meshes/torso_v0/torso_lift.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

File: trajopt/test/data/pr2.urdf (robot description, URDF)
Before this commit: robot pr2, 88 links, 87 joints
Links:
- link base_link: geometry collision mesh filename=package://trajopt/test/data/pr2/meshes/base_v0/base_L.stl; visual mesh filename=package://trajopt/test/data/pr2/meshes/base_v0/base.dae
- link bl_caster_l_wheel_link: geometry collision cylinder length=0.034 radius=0.074792; visual mesh filename=package://trajopt/test/data/pr2/meshes/base_v0/wheel.dae
- link bl_caster_r_wheel_link: geometry collision cylinder length=0.034 radius=0.074792; visual mesh filename=package://trajopt/test/data/pr2/meshes/base_v0/wheel.dae
- link bl_caster_rotation_link: geometry collision mesh filename=package://trajopt/test/data/pr2/meshes/base_v0/caster_L.stl; visual mesh filename=package://trajopt/test/data/pr2/meshes/base_v0/caster.stl
- link br_caster_l_wheel_link: geometry collision cylinder length=0.034 radius=0.074792; visual mesh filename=package://trajopt/test/data/pr2/meshes/base_v0/wheel.dae
- link br_caster_r_wheel_link: geometry collision cylinder length=0.034 radius=0.074792; visual mesh filename=package://trajopt/test/data/pr2/meshes/base_v0/wheel.dae
- link br_caster_rotation_link: geometry collision mesh filename=package://trajopt/test/data/pr2/meshes/base_v0/caster_L.stl; visual mesh filename=package://trajopt/test/data/pr2/meshes/base_v0/caster.stl
- link fl_caster_l_wheel_link: geometry collision cylinder length=0.034 radius=0.074792; visual mesh filename=package://trajopt/test/data/pr2/meshes/base_v0/wheel.dae
- link fl_caster_r_wheel_link: geometry collision cylinder length=0.034 radius=0.074792; visual mesh filename=package://trajopt/test/data/pr2/meshes/base_v0/wheel.dae
- link fl_caster_rotation_link: geometry collision mesh filename=package://trajopt/test/data/pr2/meshes/base_v0/caster_L.stl; visual mesh filename=package://trajopt/test/data/pr2/meshes/base_v0/caster.stl
- link fr_caster_l_wheel_link: geometry collision cylinder length=0.034 radius=0.074792; visual mesh filename=package://trajopt/test/data/pr2/meshes/base_v0/wheel.dae
- link fr_caster_r_wheel_link: geometry collision cylinder length=0.034 radius=0.074792; visual mesh filename=package://trajopt/test/data/pr2/meshes/base_v0/wheel.dae
- link fr_caster_rotation_link: geometry collision mesh filename=package://trajopt/test/data/pr2/meshes/base_v0/caster_L.stl; visual mesh filename=package://trajopt/test/data/pr2/meshes/base_v0/caster.stl
- link head_pan_link: geometry collision mesh filename=package://trajopt/test/data/pr2/meshes/head_v0/head_pan_L.s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; visual mesh filename=package://trajopt/test/data/pr2/meshes/head_v0/head_pan.dae
- link head_tilt_link: geometry collision mesh filename=package://trajopt/test/data/pr2/meshes/head_v0/head_tilt_L.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; visual mesh filename=package://trajopt/test/data/pr2/meshes/head_v0/head_tilt.dae
- link l_elbow_flex_link: geometry collision mesh filename=package://trajopt/test/data/pr2/meshes/upper_arm_v0/elbow_f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; visual mesh filename=package://trajopt/test/data/pr2/meshes/upper_arm_v0/elbow_f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
- link l_forearm_link: geometry collision mesh filename=package://trajopt/test/data/pr2/meshes/forearm_v0/forearm.s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; visual mesh filename=package://trajopt/test/data/pr2/meshes/forearm_v0/forearm.d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
- link l_forearm_roll_link: geometry collision mesh filename=package://trajopt/test/data/pr2/meshes/upper_arm_v0/forearm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; visual mesh filename=package://trajopt/test/data/pr2/meshes/upper_arm_v0/forearm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
- link l_gripper_l_finger_link: geometry collision mesh filename=package://trajopt/test/data/pr2/meshes/gripper_v0/l_finger.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; visual mesh filename=package://trajopt/test/data/pr2/meshes/gripper_v0/l_finger.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
- link l_gripper_l_finger_tip_link: geometry collision mesh filename=package://trajopt/test/data/pr2/meshes/gripper_v0/l_finger_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; visual mesh filename=package://trajopt/test/data/pr2/meshes/gripper_v0/l_finger_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
- link l_gripper_palm_link: geometry collision mesh filename=package://trajopt/test/data/pr2/meshes/gripper_v0/gripper_p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; visual mesh filename=package://trajopt/test/data/pr2/meshes/gripper_v0/gripper_p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
- link l_gripper_r_finger_link: geometry collision mesh filename=package://trajopt/test/data/pr2/meshes/gripper_v0/l_finger.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; visual mesh filename=package://trajopt/test/data/pr2/meshes/gripper_v0/l_finger.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
- link l_gripper_r_finger_tip_link: geometry collision mesh filename=package://trajopt/test/data/pr2/meshes/gripper_v0/l_finger_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; visual mesh filename=package://trajopt/test/data/pr2/meshes/gripper_v0/l_finger_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
- link l_shoulder_lift_link: geometry collision mesh filename=package://trajopt/test/data/pr2/meshes/shoulder_v0/shoulder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; visual mesh filename=package://trajopt/test/data/pr2/meshes/shoulder_v0/shoulder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
- link l_shoulder_pan_link: geometry collision mesh filename=package://trajopt/test/data/pr2/meshes/shoulder_v0/shoulder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; visual mesh filename=package://trajopt/test/data/pr2/meshes/shoulder_v0/shoulder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
- link l_upper_arm_link: geometry collision mesh filename=package://trajopt/test/data/pr2/meshes/upper_arm_v0/upper_a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; visual mesh filename=package://trajopt/test/data/pr2/meshes/upper_arm_v0/upper_a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
- link l_upper_arm_roll_link: geometry collision mesh filename=package://trajopt/test/data/pr2/meshes/shoulder_v0/upper_ar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; visual mesh filename=package://trajopt/test/data/pr2/meshes/shoulder_v0/upper_ar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
- link l_wrist_flex_link: geometry collision mesh filename=package://trajopt/test/data/pr2/meshes/forearm_v0/wrist_fle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; visual mesh filename=package://trajopt/test/data/pr2/meshes/forearm_v0/wrist_fle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
- link l_wrist_roll_link: geometry collision mesh filename=package://trajopt/test/data/pr2/meshes/forearm_v0/wrist_rol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; visual mesh filename=package://trajopt/test/data/pr2/meshes/forearm_v0/wrist_rol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
- link laser_tilt_mount_link: geometry collision mesh filename=package://trajopt/test/data/pr2/meshes/tilting_laser_v0/til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; visual mesh filename=package://trajopt/test/data/pr2/meshes/tilting_laser_v0/til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
- link r_elbow_flex_link: geometry collision mesh filename=package://trajopt/test/data/pr2/meshes/upper_arm_v0/elbow_f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; visual mesh filename=package://trajopt/test/data/pr2/meshes/upper_arm_v0/elbow_f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
- link r_forearm_link: geometry collision mesh filename=package://trajopt/test/data/pr2/meshes/forearm_v0/forearm.s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; visual mesh filename=package://trajopt/test/data/pr2/meshes/forearm_v0/forearm.d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
- link r_forearm_roll_link: geometry collision mesh filename=package://trajopt/test/data/pr2/meshes/upper_arm_v0/forearm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; visual mesh filename=package://trajopt/test/data/pr2/meshes/upper_arm_v0/forearm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
- link r_gripper_l_finger_link: geometry collision mesh filename=package://trajopt/test/data/pr2/meshes/gripper_v0/l_finger.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; visual mesh filename=package://trajopt/test/data/pr2/meshes/gripper_v0/l_finger.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
- link r_gripper_l_finger_tip_link: geometry collision mesh filename=package://trajopt/test/data/pr2/meshes/gripper_v0/l_finger_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; visual mesh filename=package://trajopt/test/data/pr2/meshes/gripper_v0/l_finger_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
- link r_gripper_palm_link: geometry collision mesh filename=package://trajopt/test/data/pr2/meshes/gripper_v0/gripper_p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; visual mesh filename=package://trajopt/test/data/pr2/meshes/gripper_v0/gripper_p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
- link r_gripper_r_finger_link: geometry collision mesh filename=package://trajopt/test/data/pr2/meshes/gripper_v0/l_finger.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; visual mesh filename=package://trajopt/test/data/pr2/meshes/gripper_v0/l_finger.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
- link r_gripper_r_finger_tip_link: geometry collision mesh filename=package://trajopt/test/data/pr2/meshes/gripper_v0/l_finger_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; visual mesh filename=package://trajopt/test/data/pr2/meshes/gripper_v0/l_finger_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
- link r_shoulder_lift_link: geometry collision mesh filename=package://trajopt/test/data/pr2/meshes/shoulder_v0/shoulder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; visual mesh filename=package://trajopt/test/data/pr2/meshes/shoulder_v0/shoulder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
- link r_shoulder_pan_link: geometry collision mesh filename=package://trajopt/test/data/pr2/meshes/shoulder_v0/shoulder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; visual mesh filename=package://trajopt/test/data/pr2/meshes/shoulder_v0/shoulder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
- link r_upper_arm_link: geometry collision mesh filename=package://trajopt/test/data/pr2/meshes/upper_arm_v0/upper_a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; visual mesh filename=package://trajopt/test/data/pr2/meshes/upper_arm_v0/upper_a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
- link r_upper_arm_roll_link: geometry collision mesh filename=package://trajopt/test/data/pr2/meshes/shoulder_v0/upper_ar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; visual mesh filename=package://trajopt/test/data/pr2/meshes/shoulder_v0/upper_ar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
- link r_wrist_flex_link: geometry collision mesh filename=package://trajopt/test/data/pr2/meshes/forearm_v0/wrist_fle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; visual mesh filename=package://trajopt/test/data/pr2/meshes/forearm_v0/wrist_fle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
- link r_wrist_roll_link: geometry collision mesh filename=package://trajopt/test/data/pr2/meshes/forearm_v0/wrist_rol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; visual mesh filename=package://trajopt/test/data/pr2/meshes/forearm_v0/wrist_rol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
- link torso_lift_link: geometry collision mesh filename=package://trajopt/test/data/pr2/meshes/torso_v0/torso_lift_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; visual mesh filename=package://trajopt/test/data/pr2/meshes/torso_v0/torso_lift.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
